Commit message: UPDATE: uvc1_gazebo and Re-organized Folder Structure

File: src/uvc1_gazebo/urdf/uvc1_virofighter.urdf (robot description, URDF)
Before this commit: robot uvc1_virofighter, 30 links, 29 joints
Joints:
- joint camera_fisheye_front_joint: origin xyz=0.07 0 1.845 rpy=0 0.2269 -0.0255 -> xyz=0.07 0 1.845 rpy=0 0.628 -0.0255
